File: kintsugi.kicad_pcb (KiCad board)
At the start: 2 copper layers, 304.8 x 95.3 mm, 164 parts, among them J1 Conn_01x04, SW1 Rotary_Encoder_Switch, U1 Elite-C

Commit message: Routing started
Began routing rows and columns
Parts:
- D1, D10, D11, D12, D13, D14, D15, D16, D17, D18, D19, D2, D20, D21, D22, D23, D24, D25, D26, D27, D28, D29, D3, D30, D31, D32, D33, D34, D35, D36, D37, D38, D39, D4, D40, D41, D42, D43, D44, D45, D46, D47, D48, D49, D5, D50, D51, D52, D53, D54, D55, D56, D57, D58, D59, D6, D60, D61, D62, D63, D64, D65, D7, D8, D9: footprint Diode_THT:D_DO-35_SOD27_P7.62mm_Horizontal -> Keebio-Parts:Diode-dual-onesided
- moved C16 278.0 mm to (333.2, 94.1)
- moved D28 260.5 mm to (319.0, 58.2), turned to 180 degrees
- moved D13 253.4 mm to (285.9, 39.1), turned to 180 degrees
- moved C8 251.2 mm to (306.6, 56.0)
- moved D65 240.2 mm to (342.8, 115.3), turned to 180 degrees
- moved D26 236.9 mm to (276.1, 58.2), turned to 180 degrees
- moved D66 226.7 mm to (66.7, 40.9)
- moved D2 222.7 mm to (76.3, 39.1), turned to 180 degrees
- moved D7 221.4 mm to (171.6, 39.1), turned to 180 degrees
- moved C15 220.8 mm to (261.9, 94.0)
- moved D72 219.5 mm to (228.3, 59.9)
- moved D56 211.4 mm to (342.8, 96.3), turned to 180 degrees
- moved D53 205.9 mm to (271.3, 96.3), turned to 180 degrees
- moved D14 205.3 mm to (314.3, 39.1), turned to 180 degrees
- moved D73 204.2 mm to (306.6, 60.1)
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Routing:
- net ROW0: track 0.00 -> 27.1 mm
- net Net-(D8-Pad2): track 0.00 -> 13.1 mm
- net Net-(D9-Pad2): track 0.00 -> 13.1 mm
- net Net-(D13-Pad2): track 0.00 -> 13.0 mm
- net Net-(D14-Pad2): track 0.00 -> 13.0 mm
- net Net-(D10-Pad2): track 0.00 -> 12.9 mm
- net Net-(D11-Pad2): track 0.00 -> 12.9 mm
- net Net-(D4-Pad2): track 0.00 -> 12.9 mm
- net Net-(D1-Pad2): track 0.00 -> 12.9 mm
- net Net-(D3-Pad2): track 0.00 -> 12.8 mm
- net Net-(D6-Pad2): track 0.00 -> 12.8 mm
- net Net-(D5-Pad2): track 0.00 -> 12.7 mm
- net Net-(D7-Pad2): track 0.00 -> 12.7 mm
- net Net-(D12-Pad2): track 0.00 -> 12.7 mm
- net Net-(D2-Pad2): track 0.00 -> 12.6 mm

Commit message: Columns and rows connected
Switches connected to their respective row and column
Parts:
- moved D1 0.26 mm to (57.0, 39.1)
- moved D7 0.26 mm to (171.3, 39.1)
- moved D11 0.26 mm to (247.5, 39.1)
- moved D12 0.25 mm to (266.6, 39.1)
- moved D8 0.25 mm to (190.4, 39.1)
- moved D2 0.25 mm to (76.1, 39.1)
- moved D6 0.25 mm to (152.3, 39.1)
- moved D4 0.21 mm to (114.2, 39.1)
- moved D10 0.21 mm to (228.5, 39.1)
- moved D13 0.21 mm to (285.7, 39.1)
- moved D3 0.21 mm to (95.2, 39.1)
- moved D5 0.21 mm to (133.3, 39.1)
- moved D9 0.21 mm to (209.5, 39.1)
- moved D17 0.13 mm to (104.6, 58.2)
- moved D16 0.09 mm to (85.6, 58.2)
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Connections:
- U1 pad 10: Net-(U1-Pad10) -> ULED
- U1 pad 13: Net-(U1-Pad13) -> ROW1
- U1 pad 19: ENCB -> Net-(U1-Pad19)
- U1 pad 20: ENCA -> Net-(U1-Pad20)
- U1 pad 24: ULED -> ROW0
- U1 pad 25: Net-(U1-Pad25) -> ENCB
- U1 pad 26: Net-(U1-Pad26) -> ENCA
- U1 pad 27: Net-(U1-Pad27) -> ROW4
- U1 pad 28: Net-(U1-Pad28) -> ROW3
- U1 pad 29: Net-(U1-Pad29) -> ROW2
Routing:
- net ROW3: track 0.00 -> 381.6 mm, vias 0 -> 4
- net ROW4: track 0.00 -> 381.1 mm, vias 0 -> 2
- net ROW2: track 0.00 -> 350.0 mm
- net ROW1: track 0.00 -> 343.5 mm, vias 0 -> 1
- net ROW0: track 27.1 -> 345.4 mm
- net COL11: track 0.00 -> 117.6 mm, vias 0 -> 5
- net COL10: track 0.00 -> 111.6 mm, vias 0 -> 5
- net COL6: track 0.00 -> 108.1 mm, vias 0 -> 5
- net COL2: track 0.00 -> 104.5 mm, vias 0 -> 5
- net COL0: track 0.00 -> 102.0 mm, vias 0 -> 5
- net COL1: track 0.00 -> 100.9 mm, vias 0 -> 5
- net COL13: track 0.00 -> 98.3 mm, vias 0 -> 7
- net COL12: track 0.00 -> 97.3 mm, vias 0 -> 3
- net COL7: track 0.00 -> 78.9 mm, vias 0 -> 4
- net COL8: track 0.00 -> 78.3 mm, vias 0 -> 4
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Other:
- board size 304.8 x 95.3 mm -> 308 x 95.2 mm
- net class Power added: clearance 0.2, trace_width 0.381, via_dia 0.8, via_drill 0.4

Commit message: Deleted old routing
Fresh start
Routing:
- net ROW3: track 381.6 -> 0.00 mm, vias 4 -> 0
- net ROW4: track 381.1 -> 0.00 mm, vias 2 -> 0
- net ROW2: track 350.0 -> 0.00 mm
- net ROW0: track 345.4 -> 0.00 mm
- net ROW1: track 343.5 -> 0.00 mm, vias 1 -> 0
- net COL11: track 117.6 -> 0.00 mm, vias 5 -> 0
- net COL10: track 111.6 -> 0.00 mm, vias 5 -> 0
- net COL6: track 108.1 -> 0.00 mm, vias 5 -> 0
- net COL2: track 104.5 -> 0.00 mm, vias 5 -> 0
- net COL0: track 102.0 -> 0.00 mm, vias 5 -> 0
- net COL1: track 100.9 -> 0.00 mm, vias 5 -> 0
- net COL13: track 98.3 -> 0.00 mm, vias 7 -> 0
- net COL12: track 97.3 -> 0.00 mm, vias 3 -> 0
- net COL7: track 78.9 -> 0.00 mm, vias 4 -> 0
- net COL8: track 78.3 -> 0.00 mm, vias 4 -> 0
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
Commit message: Routed rows and first three columns
Began routing the new pcb.
Parts:
- moved D28 0.12 mm to (318.9, 58.2)
Connections:
- D10 pad 1: ROW0 -> ROW5
- D11 pad 1: ROW0 -> ROW5
- D12 pad 1: ROW0 -> ROW5
- D13 pad 1: ROW0 -> ROW5
- D14 pad 1: ROW0 -> ROW5
- D22 pad 1: ROW1 -> ROW6
- D23 pad 1: ROW1 -> ROW6
- D24 pad 1: ROW1 -> ROW6
- D25 pad 1: ROW1 -> ROW6
- D26 pad 1: ROW1 -> ROW6
- D27 pad 1: ROW1 -> ROW6
- D28 pad 1: ROW1 -> ROW6
- D36 pad 1: ROW2 -> ROW7
- D37 pad 1: ROW2 -> ROW7
- D38 pad 1: ROW2 -> ROW7
- D39 pad 1: ROW2 -> ROW7
- D40 pad 1: ROW2 -> ROW7
- D41 pad 1: ROW2 -> ROW7
- D42 pad 1: ROW2 -> ROW7
- D50 pad 1: ROW3 -> ROW8
- D51 pad 1: ROW3 -> ROW8
- D52 pad 1: ROW3 -> ROW8
- D53 pad 1: ROW3 -> ROW8
- D54 pad 1: ROW3 -> ROW8
- D55 pad 1: ROW3 -> ROW8
- D56 pad 1: ROW3 -> ROW8
- D61 pad 1: ROW4 -> ROW9
- D62 pad 1: ROW4 -> ROW9
- D63 pad 1: ROW4 -> ROW9
- D64 pad 1: ROW4 -> ROW9
- D65 pad 1: ROW4 -> ROW9
- D8 pad 1: ROW0 -> ROW5
- D9 pad 1: ROW0 -> ROW5
- MX10 pad 1: COL9 -> COL2
- MX11 pad 1: COL10 -> COL3
- MX12 pad 1: COL11 -> COL4
- MX13 pad 1: COL12 -> COL5
- MX14 pad 1: COL13 -> COL6
- MX22 pad 1: COL7 -> COL0
- MX23 pad 1: COL8 -> COL1
- MX24 pad 1: COL9 -> COL2
- MX25 pad 1: COL10 -> COL3
- MX26 pad 1: COL11 -> COL4
- MX27 pad 1: COL12 -> COL5
- MX28 pad 1: COL13 -> COL6
- MX36 pad 1: COL7 -> COL0
- MX37 pad 1: COL8 -> COL1
- MX38 pad 1: COL9 -> COL2
- MX39 pad 1: COL10 -> COL3
- MX40 pad 1: COL11 -> COL4
- MX41 pad 1: COL13 -> COL5
- MX49 pad 1: COL7 -> COL0
- MX50 pad 1: COL8 -> COL1
- MX51 pad 1: COL9 -> COL2
- MX52 pad 1: COL10 -> COL3
- MX53 pad 1: COL11 -> COL4
- MX54 pad 1: COL13 -> COL5
- MX55 pad 1: COL14 -> COL6
- MX60 pad 1: COL10 -> COL2
- MX61 pad 1: COL11 -> COL3
- MX62 pad 1: COL12 -> COL4
- MX63 pad 1: COL13 -> COL5
- MX64 pad 1: COL14 -> COL6
- MX8 pad 1: COL7 -> COL0
- MX9 pad 1: COL8 -> COL1
- SW1 pad S2: COL14 -> COL6
Routing:
- net COL2: track 0.00 -> 355.2 mm, vias 0 -> 10
- net COL1: track 0.00 -> 332.0 mm, vias 0 -> 9
- net COL0: track 0.00 -> 319.9 mm, vias 0 -> 9
- net ROW7: track 0.00 -> 145.3 mm, vias 0 -> 2
- net ROW8: track 0.00 -> 143.4 mm, vias 0 -> 4
- net ROW3: track 0.00 -> 142.3 mm
- net ROW5: track 0.00 -> 140.3 mm, vias 0 -> 4
- net ROW2: track 0.00 -> 136.4 mm, vias 0 -> 4
- net ROW1: track 0.00 -> 134.1 mm, vias 0 -> 4
- net ROW6: track 0.00 -> 133.8 mm, vias 0 -> 4
- net ROW0: track 0.00 -> 129.4 mm, vias 0 -> 4
- net ROW4: track 0.00 -> 129.4 mm
- net ROW9: track 0.00 -> 102.8 mm
- net Net-(D52-Pad2): track 0.00 -> 12.4 mm
- net Net-(D15-Pad2): track 0.00 -> 12.4 mm
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
Commit message: Re-routed rows, cols, oled and encoder
Routed for the third time the board, rows in front, cols in back.
Routing:
- net COL6: track 0.00 -> 350.3 mm, vias 0 -> 2
- net COL4: track 0.00 -> 349.1 mm
- net COL5: track 0.00 -> 342.9 mm, vias 0 -> 2
- net COL3: track 0.00 -> 303.0 mm, vias 0 -> 2
- net GND: track 0.00 -> 69.6 mm, vias 0 -> 1
- net VCC: track 0.00 -> 37.8 mm
- net SDA: track 0.00 -> 30.0 mm
- net COL2: track 355.2 -> 327.0 mm, vias 10 -> 2
- net SCL: track 0.00 -> 28.0 mm
- net ENCA: track 0.00 -> 22.5 mm
- net COL1: track 332.0 -> 312.3 mm, vias 9 -> 2
- net ENCB: track 0.00 -> 15.0 mm
- net COL0: track 319.9 -> 323.6 mm, vias 9 -> 0
- net ROW1: track 134.1 -> 132.8 mm, vias 4 -> 0
- net ROW0: track 129.4 -> 128.5 mm, vias 4 -> 0
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
Commit message: Began routing leds
Started with the underglows routing
Parts:
- moved D70 233.6 mm to (307.2, 59.9), turned to 180 degrees
- moved C5 233.6 mm to (307.2, 56.0)
- moved D73 232.9 mm to (73.7, 59.9), turned to 180 degrees
- moved C8 232.9 mm to (73.7, 56.0)
- moved D72 76.5 mm to (151.9, 59.9), turned to 180 degrees
- moved C7 76.3 mm to (152.0, 56.0)
- moved D71 75.8 mm to (228.1, 59.9), turned to 180 degrees
- moved C6 75.8 mm to (228.2, 56.0)
- moved D68 0.52 mm to (218.6, 40.9), turned to 180 degrees
- moved C2 0.51 mm to (142.4, 36.8)
- moved D67 0.51 mm to (142.4, 40.9), turned to 180 degrees
- moved D66 0.51 mm to (66.2, 40.9), turned to 180 degrees
- moved C3 0.40 mm to (218.7, 37.0)
- moved C1 0.25 mm to (66.2, 36.8), turned to 0 degrees
- turned D69 to 180 degrees
Routing:
- net GND: track 69.6 -> 530.0 mm, vias 1 -> 8
- net VCC: track 37.8 -> 468.1 mm, vias 0 -> 7
- net Net-(D70-Pad2): track 0.00 -> 104.3 mm, vias 0 -> 2
- net Net-(D71-Pad2): track 0.00 -> 96.3 mm, vias 0 -> 2
- net Net-(D66-Pad2): track 0.00 -> 79.4 mm, vias 0 -> 2
- net Net-(D67-Pad2): track 0.00 -> 78.9 mm, vias 0 -> 2
- net Net-(D68-Pad2): track 0.00 -> 74.5 mm, vias 0 -> 2
- net Net-(D69-Pad2): track 0.00 -> 20.2 mm
- net COL2: track 327.0 -> 325.0 mm

Commit message: Routed first 5 rows
Finished routing leds and first 5 rows
Parts:
- moved D81 262.7 mm to (70.9, 111.5), turned to 180 degrees
- moved C16 262.6 mm to (71.0, 107.6)
- moved C13 262.1 mm to (333.0, 94.1)
- moved D78 261.7 mm to (332.9, 98.0), turned to 180 degrees
- moved D80 96.4 mm to (165.5, 102.9), turned to 180 degrees
- moved D79 95.9 mm to (261.2, 98.0), turned to 180 degrees
- moved C14 9.27 mm to (165.5, 98.9)
- moved D74 2.01 mm to (76.6, 77.1), turned to 180 degrees
- moved C9 1.97 mm to (76.6, 73.0)
- moved C15 0.54 mm to (261.3, 94.1)
- moved C10 0.38 mm to (156.6, 75.1)
- moved C11 0.38 mm to (232.9, 75.1)
- moved D75 0.38 mm to (156.6, 79.0), turned to 180 degrees
- moved D76 0.38 mm to (232.9, 79.0), turned to 180 degrees
- moved C12 0.25 mm to (310.5, 87.6)
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Connections:
- U1 pad 10: ULED -> ROW1
- U1 pad 13: ROW1 -> Net-(U1-Pad13)
- U1 pad 2: Net-(U1-Pad2) -> ROW5
- U1 pad 27: ROW4 -> Net-(U1-Pad27)
- U1 pad 28: ROW3 -> Net-(U1-Pad28)
- U1 pad 29: ROW2 -> Net-(U1-Pad29)
- U1 pad 7: Net-(U1-Pad7) -> ROW4
- U1 pad 8: Net-(U1-Pad8) -> ROW3
- U1 pad 9: Net-(U1-Pad9) -> ROW2
Routing:
- net VCC: track 468.1 -> 1240.9 mm, vias 7 -> 17
- net GND: track 530.0 -> 1200.5 mm, vias 8 -> 19
- net ROW4: track 129.4 -> 545.3 mm
- net ROW3: track 142.3 -> 549.5 mm
- net ROW2: track 135.6 -> 519.1 mm
- net ROW1: track 132.8 -> 492.6 mm
- net ROW0: track 128.5 -> 434.6 mm
- net Net-(D80-Pad2): track 0.00 -> 120.6 mm, vias 0 -> 2
- net Net-(D79-Pad2): track 0.00 -> 119.2 mm, vias 0 -> 2
- net Net-(D72-Pad2): track 0.00 -> 109.5 mm, vias 0 -> 2
- net Net-(D78-Pad2): track 0.00 -> 90.1 mm, vias 0 -> 2
- net Net-(D76-Pad2): track 0.00 -> 87.2 mm, vias 0 -> 2
- net Net-(D74-Pad2): track 0.00 -> 84.1 mm, vias 0 -> 2
- net Net-(D75-Pad2): track 0.00 -> 81.1 mm, vias 0 -> 2
- net Net-(D77-Pad2): track 0.00 -> 74.4 mm
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
Commit message: Finished routing and gnd fill
First revision completed, waiting for review
Connections:
- U1 pad 11: Net-(U1-Pad11) -> ROW9
- U1 pad 12: Net-(U1-Pad12) -> ROW8
- U1 pad 13: Net-(U1-Pad13) -> COL5
- U1 pad 14: Net-(U1-Pad14) -> COL4
- U1 pad 15: Net-(U1-Pad15) -> COL3
- U1 pad 16: Net-(U1-Pad16) -> COL2
- U1 pad 17: Net-(U1-Pad17) -> COL1
- U1 pad 18: Net-(U1-Pad18) -> COL0
- U1 pad 19: Net-(U1-Pad19) -> ROW7
- U1 pad 20: Net-(U1-Pad20) -> ROW6
- U1 pad 28: Net-(U1-Pad28) -> ULED
- U1 pad 29: Net-(U1-Pad29) -> COL6
Routing:
- net ULED: track 0.00 -> 337.8 mm, vias 0 -> 1
- net COL0: track 323.6 -> 484.6 mm, vias 0 -> 1
- net COL1: track 312.3 -> 463.7 mm, vias 2 -> 4
- net COL2: track 325.0 -> 441.1 mm, vias 2 -> 3
- net COL3: track 302.7 -> 400.7 mm, vias 2 -> 3
- net COL4: track 349.1 -> 428.5 mm, vias 0 -> 1
- net ROW9: track 102.8 -> 181.2 mm
- net COL5: track 342.6 -> 402.5 mm, vias 2 -> 3
- net ROW8: track 142.6 -> 199.8 mm
- net ROW7: track 145.1 -> 184.5 mm
- net ROW6: track 133.0 -> 168.8 mm
- net COL6: track 350.3 -> 376.5 mm
- net VCC: track 1240.9 -> 1242.0 mm
- added copper zone on B.Cu, net GND
- added copper zone on F.Cu, net GND
