File: kintsugi.kicad_pcb (KiCad board)
At the start: 2 copper layers, 308 x 95.2 mm, 164 parts, among them J1 Conn_01x04, SW1 Rotary_Encoder_Switch, U1 Elite-C

Commit message: Added silkscreen logos
Almost there
Parts:
- added G***: LOGO, logos:LogoKC1, B.Cu at (216.2, 107.2)
Routing:
- net GND: vias 19 -> 31
Other:
- board text added: "Kintsugi rev. 1.0 Designed by ADPenrose/Arturo Avila"

Commit message: Gerber files generated
I think this is where it ends
Parts:
- moved G*** 0.13 mm to (216.0, 107.2)
Other:
- board text added: "Kintsugi rev. 1.0 Designed by ADPenrose/Arturo Avila For more information, go to https://github.com /ADPenrose/kintsugi_keeb"
- board text added: "Made with love by a mexican, for the whole keyboard community <3"
- board text removed: "Kintsugi rev. 1.0 Designed by ADPenrose/Arturo Avila"

Commit message: Case
Added proto case files
Parts:
- removed G***: LOGO, logos:LogoKC1
